File: hardware/board/main.kicad_pcb (KiCad board)
At the start: 4 copper layers, 44.5 x 34.9 mm, 55 parts, among them Q1 DMG6968UDM, U1 AP2112K, U11 ATSAMD21E18A-A, U2 MCP73831, U3 AP9101CK6

Commit message: Update board files
Added extra pad, so the battery can be connected without removing the protection circuit
Parts:
- added TP10: ~, main:TestPoint_Pad_2.0x2.5mm, B.Cu at (31.1, 62.2)
Other:
- board text added: "+ -"
- board text added: "Eclair Rev.C - mateusznowak.dev/eclair"
- board text added: "Li-Po battery 25x15mm max 30mA chg.cur. Do not populate Q1,U3,C4,R3,R4"
- board text added: "NC"
- board text removed: "+"
- board text removed: "-"
- board text removed: "Eclair Rev.B - mateusznowak.dev/eclair"
