File: hardware/board/main.kicad_pcb (KiCad board)
At the start: 4 copper layers, 44.5 x 34.9 mm, 56 parts, among them Q1 DMG6968UDM, U1 AP2112K, U11 ATSAMD21E18A-A, U2 MCP73831, U3 AP9101CK6

Commit message: Update project name to improve discoverability
Other:
- board text added: "EclairM0 Rev.C - mateusznowak.dev/eclair"
- board text removed: "Eclair Rev.C - mateusznowak.dev/eclair"
Changed lines of the file:
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@@
 		)
 	)
-	(gr_text "Eclair Rev.C - mateusznowak.dev/eclair"
+	(gr_text "EclairM0 Rev.C - mateusznowak.dev/eclair"
 		(at 50.8 66.3575 0)
 		(layer "B.SilkS")

Commit message: Change battery measurement circuit
Use 22K / 5.1K voltage divider and fixed 1V reference. This should work correctly even if system voltage goes below 3.3V.
Parts:
- R51: value 33K -> 22K
- R52: value 33K -> 5.1K
Changed lines of the file:
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@@
 			)
 		)
-		(property "Value" "33K"
+		(property "Value" "22K"
 			(at 0 -1.65 90)
 			(layer "B.Fab")
@@
 			)
 		)
-		(property "Value" "33K"
+		(property "Value" "5.1K"
 			(at 0 -1.65 90)
 			(layer "B.Fab")

Commit message: Replace Li-Po battery with rechargeable coin battery
Charging circuit has been moved closer to the USB. The slide switch is now mounted on the bottom layer. Battery protection circuit is removed due to lack of space. Updated for KiCad 9.0.2, optimized traces, run ERC/DRC.
Parts:
- removed C4: 1u, Capacitor_SMD:C_0805_2012Metric
- removed the J1 at (37.5, 62.2)
- removed Q1: DMG6968UDM, Package_TO_SOT_SMD:SOT-23-6
- removed the R3 at (47.3, 62.9)
- removed R4: 1K, Resistor_SMD:R_0805_2012Metric
- removed TP10: ~, main:TestPoint_Pad_2.0x2.5mm
- removed U3: AP9101CK6, Package_TO_SOT_SMD:SOT-23-6
- added BT1: ~, main:BatteryHolder_MPD_BC2003_1x2032, B.Cu at (41.3, 55.2)
- D1, S1: moved to B.Cu
- R1: renamed from R2; value 33K -> 68K
- moved C3 19.8 mm to (35.9, 39.7), turned to 90 degrees
- moved R1 17.5 mm to (36.5, 42.9), turned to 0 degrees
- moved U2 14.7 mm to (39.4, 39.7), turned to 0 degrees
- moved D2 14.3 mm to (42.5, 35.2), turned to 0 degrees
- moved C1 8.80 mm to (42.9, 39.7)
- moved D1 4.32 mm to (36.2, 35.2), turned to 180 degrees
- turned S1 to 90 degrees
- renumbered J2 to J1, R5 to R2, R6 to R3
Connections:
- S1 pad 1: Net-(D1-A) -> +BATT
- S1 pad 3: +BATT -> Net-(D1-A)
Routing:
- net +BATT: track 55.9 -> 14.1 mm, vias 2 -> 0
- net -BATT: track 22.7 -> 0.00 mm
- net VBUS: track 46.1 -> 33.0 mm, vias 4 -> 2
- net Net-(D2-A): track 26.9 -> 16.0 mm
- net Net-(U3-VDD): track 10.2 -> 0.00 mm
- net Net-(U3-VM): track 4.60 -> 0.00 mm
- net Net-(Q1-G2): track 3.44 -> 0.00 mm
- net Net-(Q1-G1): track 3.44 -> 0.00 mm
- net Net-(U2-PROG): track 3.40 -> 4.46 mm
- net /COL1: track 47.4 -> 46.4 mm
- net /COL2: track 38.9 -> 38.0 mm
- net /SWCLK: track 3.23 -> 2.72 mm
- net GND: vias 6 -> 11
Other:
- board text added: "3V"
- board text added: "5V"
- board text added: "LED"
- board text added: "RST"
- board text added: "mateusznowak.dev/eclair EclairM0 Rev.D"
- board text removed: "+ -"
- board text removed: "EclairM0 Rev.C - mateusznowak.dev/eclair"
- board text removed: "G"
- board text removed: "Li-Po battery 25x15mm max 30mA chg.cur. Do not populate Q1,U3,C4,R3,R4"
- board text removed: "NC"
- board text removed: "R"
