File: hardware/board/main.kicad_sch (KiCad schematic)
At the start: 55 parts, among them Q1 DMG6968UDM, U1 AP2112K, U11 ATSAMD21E18A-A, U2 MCP73831, U3 AP9101CK6

Commit message: Update board files
Added extra pad, so the battery can be connected without removing the protection circuit
Parts:
- added TP10: ~, main:TestPoint_Pad_2.0x2.5mm, symbol Connector:TestPoint
Connections:
- net GND: now also TP10.1
Other:
- title: ECLAIR USB KEYBOARD -> ECLAIR POCKET NOTEPAD
Changed lines of the file:
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@@
 	(paper "A4")
 	(title_block
-		(title "ECLAIR USB KEYBOARD")
-		(rev "B")
+		(title "ECLAIR POCKET NOTEPAD")
+		(date "2025-04-09")
+		(rev "C")
 	)
 	(text "Microcontroller"
@@
 	(wire
 		(pts
+			(xy 254 151.13) (xy 254 157.48)
+		)
+		(stroke
+			(width 0)
+			(type default)
+		)
+	)
+	(wire
+		(pts
 			(xy 128.27 161.29) (xy 110.49 161.29)
 		)
@@
 		)
 	)
+	(label "GND"
+		(at 254 157.48 90)
+		(effects
+			(font
+				(size 1.27 1.27)
+			)
+			(justify left bottom)
+		)
+	)
 	(label "SPI_MOSI"
 		(at 261.62 81.28 270)
@@
 					(unit 1)
 				)
+			)
+		)
+	)
+	(symbol
+		(lib_id "Connector:TestPoint")
+		(at 254 151.13 0)
+		(unit 1)
+		(exclude_from_sim no)
+		(in_bom yes)
+		(on_board yes)
+		(dnp no)
+		(property "Reference" "TP10"
+			(at 252.222 145.288 0)
+			(effects
+				(font
+					(size 1.27 1.27)
+				)
+				(justify left)
+			)
+		)
+		(property "Value" "~"
+			(at 256.54 149.0979 0)
+			(effects
+				(font
+					(size 1.27 1.27)
+				)
+				(justify left)
+			)
+		)
+		(property "Footprint" "main:TestPoint_Pad_2.0x2.5mm"
+			(at 259.08 151.13 0)
+			(effects
+				(font
+					(size 1.27 1.27)
+				)
+				(hide yes)
+			)
+		)
+		(property "Datasheet" "~"
+			(at 259.08 151.13 0)
+			(effects
+				(font
+					(size 1.27 1.27)
+				)
+				(hide yes)
+			)
+		)
+		(property "Description" "test point"
+			(at 254 151.13 0)
+			(effects
+				(font
+					(size 1.27 1.27)
+				)
+				(hide yes)
+			)
+		)
+		(pin "1"
+		)
+		(instances
+			(project "main"
+				(path "/8c2a105f-a962-4917-8f56-dd50da121d32"
+					(reference "TP10")
+					(unit 1)
+				)

Commit message: Update project name to improve discoverability
Other:
- title: ECLAIR POCKET NOTEPAD -> EclairM0 Pocket Notepad
Changed lines of the file:
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@@
 	(paper "A4")
 	(title_block
-		(title "ECLAIR POCKET NOTEPAD")
+		(title "EclairM0 Pocket Notepad")
 		(date "2025-04-09")
 		(rev "C")

Commit message: Change battery measurement circuit
Use 22K / 5.1K voltage divider and fixed 1V reference. This should work correctly even if system voltage goes below 3.3V.
Parts:
- R51: value 33K -> 22K
- R52: value 33K -> 5.1K
Changed lines of the file:
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@@
 			)
 		)
-		(property "Value" "33K"
+		(property "Value" "5.1K"
 			(at 180.34 115.5699 0)
 			(effects
@@
 			)
 		)
-		(property "Value" "33K"
+		(property "Value" "22K"
 			(at 180.34 105.4099 0)
 			(effects

Commit message: Replace Li-Po battery with rechargeable coin battery
Charging circuit has been moved closer to the USB. The slide switch is now mounted on the bottom layer. Battery protection circuit is removed due to lack of space. Updated for KiCad 9.0.2, optimized traces, run ERC/DRC.
Parts:
- removed C4: 1u, Capacitor_SMD:C_0805_2012Metric, symbol Device:C_Small
- removed J1: ~, main:LP301525, symbol Connector_Generic:Conn_01x02
- removed Q1: DMG6968UDM, Package_TO_SOT_SMD:SOT-23-6, symbol Transistor_FET:DMG9926UDM
- removed R3: 1K, Resistor_SMD:R_0805_2012Metric, symbol Device:R
- removed R4: 1K, Resistor_SMD:R_0805_2012Metric, symbol Device:R_Small
- removed TP10: ~, main:TestPoint_Pad_2.0x2.5mm, symbol Connector:TestPoint
- removed U3: AP9101CK6, Package_TO_SOT_SMD:SOT-23-6, symbol Battery_Management:AP9101CK6
- added BT1: ~, main:BatteryHolder_MPD_BC2003_1x2032, symbol Device:Battery_Cell
- R1: renamed from R2; value 33K -> 68K
- renumbered J2 to J1, R5 to R2, R6 to R3
Connections:
- net +BATT: now also S1.1 (A), BT1.1 (+); no longer S1.3 (C)
- net GND: now also BT1.2 (-)
- net at D1.2 (A): now also S1.3 (C); no longer S1.1 (A)
- no-connect marks 10 -> 9
Other:
- note added: "1000/68K = 15mA chg. current (min) 1000/33K = 30mA chg. current"
- note removed: "1000/33K = 30mA chg. current"
- moved on the sheet: D1, S1
